File: clock.brd (EAGLE design)
At the start: 100 x 80 mm, 44 parts, among them J3 POWER_JACKSLT, U2 LM75A_SO8, U3 ESP8266_13

Commit message: Added a power led and some silkscreen to make the footprints for the temperature sensors more obvious
Parts:
- added D2: (no value), Sebastian:0805_LED
- added R14: 1k, Sebastian:0603
Connections:
- new net N$4: D2.A, R14.1
- net GND: now also D2.C
- net PVDD: now also R14.2
Routing:
- net PVDD: track 156.2 -> 167.4 mm
- net GND: track 302.5 -> 308.5 mm
- net N$4: track 0.00 -> 1.89 mm
Other:
- board text added: "BME280"
- board text added: "LM75A"
- board text removed: "Light"
- board text removed: "Temperature"
Changed lines of the file:
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@@
 <text x="4.2" y="27" size="1.016" layer="21" font="vector" ratio="12" rot="R90" align="top-center">Reset</text>
 <text x="6.8" y="27" size="1.016" layer="21" font="vector" ratio="12" rot="R270" align="top-center">Flash</text>
-<text x="99" y="17.65" size="1.016" layer="21" font="vector" ratio="12" rot="R180" align="center-left">5V</text>
+<text x="99" y="18.15" size="1.016" layer="21" font="vector" ratio="12" rot="R180" align="center-left">5V</text>
 <text x="11.9" y="40" size="1.016" layer="22" font="vector" ratio="12" rot="MR270" align="center">Not GND!</text>
 <text x="22.7" y="25" size="1.016" layer="21" font="vector" ratio="12" align="center">2</text>
@@
 <dimension x1="3.5" y1="3.5" x2="96.5" y2="3.5" x3="50" y3="-2.6" textsize="1.016" textratio="12" layer="51" dtype="horizontal"/>
 <dimension x1="96.5" y1="76.5" x2="96.5" y2="3.5" x3="108.9" y3="40" textsize="1.016" textratio="12" layer="51"/>
-<text x="10" y="59" size="1.016" layer="21" font="vector" ratio="12" align="center-left">Temperature</text>
-<text x="10" y="66.7" size="1.016" layer="21" font="vector" ratio="12" align="center-left">Light</text>
+<text x="10" y="59" size="1.016" layer="21" font="vector" ratio="12" align="center-left">LM75A</text>
+<text x="10" y="66.7" size="1.016" layer="21" font="vector" ratio="12" align="center-left">BME280</text>
+<wire x1="9.4" y1="60.2" x2="15.1" y2="60.2" width="0.127" layer="21"/>
+<wire x1="15.1" y1="60.2" x2="15.1" y2="57.8" width="0.127" layer="21"/>
+<wire x1="15.1" y1="57.8" x2="9.4" y2="57.8" width="0.127" layer="21"/>
+<wire x1="9.4" y1="57.8" x2="9.4" y2="60.2" width="0.127" layer="21"/>
+<wire x1="9.4" y1="67.9" x2="15.9" y2="67.9" width="0.127" layer="21"/>
+<wire x1="9.4" y1="65.5" x2="9.4" y2="67.9" width="0.127" layer="21"/>
+<wire x1="15.9" y1="65.5" x2="9.4" y2="65.5" width="0.127" layer="21"/>
+<wire x1="15.9" y1="67.9" x2="15.9" y2="65.5" width="0.127" layer="21"/>
 </plain>
 <attributes>
@@
 <element name="J6" library="Connectors" package="1X2" value="" x="35" y="63" rot="R90"/>
 <element name="J7" library="Connectors" package="1X2" value="" x="35" y="24" rot="R90"/>
+<element name="D2" library="Sebastian" package="0805_LED" value="" x="96" y="18.1" smashed="yes" rot="R270">
+<attribute name="NAME" x="92.5" y="17" size="1.016" layer="25" font="vector" ratio="12" rot="R90" align="center-left"/>
+</element>
+<element name="R14" library="Sebastian" package="0603" value="1k" x="94.2" y="18.1" smashed="yes" rot="R270">
+<attribute name="NAME" x="90.9" y="17" size="1.016" layer="25" font="vector" ratio="12" rot="R90" align="center-left"/>
+</element>
 </elements>
 <signals>
@@
 <wire x1="7" y1="64.2" x2="7" y2="64.275" width="0.254" layer="1"/>
 <wire x1="7" y1="64.275" x2="5.975" y2="65.3" width="0.254" layer="1"/>
+<contactref element="D2" pad="C"/>
+<wire x1="93.28" y1="14.58" x2="92.2" y2="14.58" width="0.254" layer="1"/>
+<wire x1="96" y1="17.2" x2="93.38" y2="14.58" width="0.254" layer="1"/>
+<wire x1="93.38" y1="14.58" x2="92.2" y2="14.58" width="0.254" layer="1"/>
 </signal>
 <signal name="PVDD">
@@
 <wire x1="28.07" y1="25.72" x2="30.12" y2="25.72" width="0.8128" layer="16"/>
 <wire x1="30.12" y1="25.72" x2="31" y2="26.6" width="0.8128" layer="16"/>
+<contactref element="R14" pad="2"/>
+<wire x1="89.2" y1="14.58935" x2="89.2" y2="9.58" width="0.254" layer="1"/>
+<wire x1="94.2" y1="17.425" x2="92.8344" y2="16.0594" width="0.254" layer="1"/>
+<wire x1="92.8344" y1="16.0594" x2="90.67005" y2="16.0594" width="0.254" layer="1"/>
+<wire x1="90.67005" y1="16.0594" x2="89.2" y2="14.58935" width="0.254" layer="1"/>
 <wire x1="32.5" y1="38" x2="33" y2="51.5" width="0" layer="19" extent="1-1"/>
 </signal>
@@
 <wire x1="35" y1="29" x2="35" y2="25.27" width="1.016" layer="16"/>
 </signal>
+<signal name="N$4">
+<contactref element="D2" pad="A"/>
+<contactref element="R14" pad="1"/>
+<wire x1="96" y1="19" x2="95.775" y2="18.775" width="0.254" layer="1"/>
+<wire x1="95.775" y1="18.775" x2="94.2" y2="18.775" width="0.254" layer="1"/>
+</signal>
 </signals>
